File: HotPlate.kicad_sch (KiCad schematic)
At the start: 37 parts, among them J1 Barrel_Jack_Switch, J2 ICSP, U1 LMT85LP

Commit message: update
Parts:
- removed D1, D2: D_Schottky, symbol Device:D_Schottky
- added SMAJ18A1: SMAJ18A, Diode_SMD:D_SOD-123, symbol Diode:ESD9B3.3ST5G
- 0.91"OLED1: footprint (none) -> Display:SSD1306-0.91-OLED-4pin-128x32
- J1: footprint Connector_BarrelJack:BarrelJack_CLIFF_FC681465S_SMT_Horizontal -> Connector_BarrelJack:BarrelJack_Horizontal
- PD1: footprint (none) -> Diode_SMD:D_SOD-123
Connections:
- net Element: now also SMAJ18A1.2 (A2)
- net GND: now also SMAJ18A1.1 (A1)
Changed lines of the file:
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@@
   (junction (at 252.73 86.106) (diameter 0) (color 0 0 0 0)
   )
+  (junction (at 226.314 20.066) (diameter 0) (color 0 0 0 0)
+  )
   (junction (at 252.73 93.726) (diameter 0) (color 0 0 0 0)
   )
@@
   (junction (at 111.76 34.036) (diameter 0) (color 0 0 0 0)
   )
-  (junction (at 225.552 20.066) (diameter 0) (color 0 0 0 0)
+  (junction (at 226.314 35.306) (diameter 0) (color 0 0 0 0)
   )
   (junction (at 170.688 28.956) (diameter 0) (color 0 0 0 0)
@@
   )
   (junction (at 38.862 78.74) (diameter 0) (color 0 0 0 0)
-  )
-  (junction (at 225.552 35.306) (diameter 0) (color 0 0 0 0)
   )
   (junction (at 246.634 20.066) (diameter 0) (color 0 0 0 0)
@@
     (stroke (width 0) (type default) (color 0 0 0 0))
   )
+  (wire (pts (xy 226.314 20.066) (xy 234.95 20.066))
+    (stroke (width 0) (type default) (color 0 0 0 0))
+  )
   (wire (pts (xy 220.472 27.432) (xy 220.472 29.972))
     (stroke (width 0) (type default) (color 0 0 0 0))
@@
     (stroke (width 0) (type default) (color 0 0 0 0))
   )
-  (wire (pts (xy 234.95 20.066) (xy 225.552 20.066))
-    (stroke (width 0) (type default) (color 0 0 0 0))
-  )
   (wire (pts (xy 40.894 64.516) (xy 40.894 73.66))
     (stroke (width 0) (type default) (color 0 0 0 0))
   )
+  (wire (pts (xy 226.314 20.066) (xy 226.314 23.368))
+    (stroke (width 0) (type default) (color 0 0 0 0))
+  )
   (wire (pts (xy 234.95 35.306) (xy 242.316 35.306))
     (stroke (width 0) (type default) (color 0 0 0 0))
@@
     (stroke (width 0) (type default) (color 0 0 0 0))
   )
-  (wire (pts (xy 225.552 35.306) (xy 220.472 35.306))
+  (wire (pts (xy 220.472 35.306) (xy 226.314 35.306))
     (stroke (width 0) (type default) (color 0 0 0 0))
   )
@@
     (stroke (width 0) (type default) (color 0 0 0 0))
   )
-  (wire (pts (xy 225.552 35.306) (xy 234.95 35.306))
-    (stroke (width 0) (type default) (color 0 0 0 0))
-  )
   (wire (pts (xy 44.45 36.576) (xy 38.608 36.576))
     (stroke (width 0) (type default) (color 0 0 0 0))
@@
     (stroke (width 0) (type default) (color 0 0 0 0))
   )
+  (wire (pts (xy 226.314 35.306) (xy 234.95 35.306))
+    (stroke (width 0) (type default) (color 0 0 0 0))
+  )
   (wire (pts (xy 30.734 38.354) (xy 30.734 41.656))
     (stroke (width 0) (type default) (color 0 0 0 0))
@@
     (stroke (width 0) (type default) (color 0 0 0 0))
   )
+  (wire (pts (xy 226.314 30.988) (xy 226.314 35.306))
+    (stroke (width 0) (type default) (color 0 0 0 0))
+  )
   (polyline (pts (xy 238.76 43.942) (xy 238.76 81.026))
     (stroke (width 0) (type default) (color 0 0 0 0))
@@
     (stroke (width 0) (type default) (color 0 0 0 0))
   )
-  (wire (pts (xy 220.726 20.066) (xy 225.552 20.066))
+  (wire (pts (xy 220.726 20.066) (xy 226.314 20.066))
     (stroke (width 0) (type default) (color 0 0 0 0))
   )
@@
     (pin "2")
   )
-  (symbol (lib_id "Device:D_Schottky") (at 225.552 23.876 90) (unit 1)
-    (in_bom yes) (on_board yes)
-    (property "Reference" "D1" (id 0) (at 227.584 23.285 90)
-      (effects (font (size 1.27 1.27)) (justify right))
-    )
-    (property "Value" "D_Schottky" (id 1) (at 223.266 18.796 90)
-      (effects (font (size 1.27 1.27)) (justify right))
-    )
-    (property "Footprint" "" (id 2) (at 225.552 23.876 0)
-      (effects (font (size 1.27 1.27)) hide)
-    )
-    (property "Datasheet" "~" (id 3) (at 225.552 23.876 0)
-      (effects (font (size 1.27 1.27)) hide)
-    )
-    (pin "1")
-    (pin "2")
-  )
   (symbol (lib_id "Connector:Barrel_Jack_Switch") (at 210.058 27.432 0) (unit 1)
     (in_bom yes) (on_board yes) (fields_autoplaced)
     (property "Reference" "J1" (id 0) (at 210.058 19.6555 0))
     (property "Value" "Barrel_Jack_Switch" (id 1) (at 210.058 22.4306 0))
-    (property "Footprint" "Connector_BarrelJack:BarrelJack_CLIFF_FC681465S_SMT_Horizontal" (id 2) (at 211.328 28.448 0)
+    (property "Footprint" "Connector_BarrelJack:BarrelJack_Horizontal" (id 2) (at 211.328 28.448 0)
       (effects (font (size 1.27 1.27)) hide)
     )
@@
       (effects (font (size 1.27 1.27)) (justify left))
     )
-    (property "Footprint" "" (id 2) (at 222.25 152.908 0)
+    (property "Footprint" "Display:SSD1306-0.91-OLED-4pin-128x32" (id 2) (at 222.25 152.908 0)
       (effects (font (size 1.27 1.27)) hide)
     )
@@
     (pin "2")
   )
+  (symbol (lib_id "Diode:ESD9B3.3ST5G") (at 226.314 27.178 90) (unit 1)
+    (in_bom yes) (on_board yes)
+    (property "Reference" "SMAJ18A1" (id 0) (at 224.79 18.796 90)
+      (effects (font (size 1.27 1.27)) (justify right))
+    )
+    (property "Value" "SMAJ18A" (id 1) (at 220.98 16.51 90)
+      (effects (font (size 1.27 1.27)) (justify right))
+    )
+    (property "Footprint" "Diode_SMD:D_SOD-123" (id 2) (at 226.314 27.178 0)
+      (effects (font (size 1.27 1.27)) hide)
+    )
+    (property "Datasheet" "https://www.onsemi.com/pub/Collateral/ESD9B-D.PDF" (id 3) (at 226.314 27.178 0)
+      (effects (font (size 1.27 1.27)) hide)
+    )
+    (pin "1")
+    (pin "2")
+  )
   (symbol (lib_id "Device:C") (at 118.364 53.086 0) (unit 1)
     (in_bom yes) (on_board yes) (fields_autoplaced)
@@
     (pin "2")
   )
-  (symbol (lib_id "Device:D_Schottky") (at 225.552 31.496 270) (unit 1)
-    (in_bom yes) (on_board yes)
-    (property "Reference" "D2" (id 0) (at 227.584 30.27 90)
-      (effects (font (size 1.27 1.27)) (justify left))
-    )
-    (property "Value" "D_Schottky" (id 1) (at 220.726 37.592 90)
-      (effects (font (size 1.27 1.27)) (justify left))
-    )
-    (property "Footprint" "" (id 2) (at 225.552 31.496 0)
-      (effects (font (size 1.27 1.27)) hide)
-    )
-    (property "Datasheet" "~" (id 3) (at 225.552 31.496 0)
-      (effects (font (size 1.27 1.27)) hide)
-    )
-    (pin "1")
-    (pin "2")
-  )
   (symbol (lib_id "Device:C") (at 45.974 78.74 90) (unit 1)
     (in_bom yes) (on_board yes)
@@
     (property "Reference" "PD1" (id 0) (at 254.508 15.494 0))
     (property "Value" "D" (id 1) (at 254.254 17.6046 0))
-    (property "Footprint" "" (id 2) (at 254.254 20.066 0)
+    (property "Footprint" "Diode_SMD:D_SOD-123" (id 2) (at 254.254 20.066 0)
       (effects (font (size 1.27 1.27)) hide)
     )
@@
   (symbol_instances
     (path "/32aba14f-43f5-4a84-9b22-b8b9f50652be"
-      (reference "0.91\"OLED1") (unit 1) (value "Conn_01x04_Female") (footprint "")
+      (reference "0.91\"OLED1") (unit 1) (value "Conn_01x04_Female") (footprint "Display:SSD1306-0.91-OLED-4pin-128x32")
     )
     (path "/eb63c3d5-07d6-4ad3-9fe3-e2c15774aca4"
@@
       (reference "Crystal1") (unit 1) (value "16Mhz") (footprint "Crystal:Crystal_SMD_5032-2Pin_5.0x3.2mm")
     )
-    (path "/26431856-1ff3-4805-9fd1-93053c250f4c"
-      (reference "D1") (unit 1) (value "D_Schottky") (footprint "")
-    )
-    (path "/97f87cca-ace2-4158-94bf-9cc9a6a22ef7"
-      (reference "D2") (unit 1) (value "D_Schottky") (footprint "")
-    )
     (path "/5bee1e88-077a-4a94-a514-403fd53dc52f"
       (reference "DNSW1") (unit 1) (value "K8-5851E-N1") (footprint "Button_Switch_Keyboard:K85851EN1")
@@
     )
     (path "/2cd8a903-0261-4f09-ba77-606d0a316220"
-      (reference "J1") (unit 1) (value "Barrel_Jack_Switch") (footprint "Connector_BarrelJack:BarrelJack_CLIFF_FC681465S_SMT_Horizontal")
+      (reference "J1") (unit 1) (value "Barrel_Jack_Switch") (footprint "Connector_BarrelJack:BarrelJack_Horizontal")
     )
     (path "/0a2bfccd-afd0-47be-ae8c-9cb2c3a84928"
@@
     )
     (path "/e2b5dd16-d649-4f0f-b4ba-dca0c7f9e14e"
-      (reference "PD1") (unit 1) (value "D") (footprint "")
+      (reference "PD1") (unit 1) (value "D") (footprint "Diode_SMD:D_SOD-123")
     )
     (path "/73478ba4-40b7-44d7-a9a1-d0599ba204db"
@@
       (reference "PR2") (unit 1) (value "1K") (footprint "Capacitor_SMD:C_1206_3216Metric_Pad1.33x1.80mm_HandSolder")
     )
+    (path "/737c3eb0-edd7-42a7-b782-07a107f00a56"
+      (reference "SMAJ18A1") (unit 1) (value "SMAJ18A") (footprint "Diode_SMD:D_SOD-123")
+    )
     (path "/5e169214-d607-4df1-a2e0-f4e16f38d5f4"
