File: ESP32 NEXTION/HotPlate.kicad_pcb (KiCad board)
At the start: 2 copper layers, 170.7 x 111.2 mm, 63 parts, among them J1 Barrel_Jack_Switch, J11 Conn_01x04_Male, J2 Conn_01x08_Male

Commit message: revision 1.2
Parts:
- TC2: moved to B.Cu
- moved REF** 65.9 mm to (29.6, 105.3)
- moved TC1 44.9 mm to (28.2, 4.97), turned to 0 degrees
- moved LMT1 35.0 mm to (27.2, 10.6), turned to 0 degrees
- moved G*** 15.6 mm to (96.2, 16.2)
- moved G*** 15.6 mm to (96.3, 15.6)
- moved G*** 12.0 mm to (47.2, 12.6)
- moved G*** 11.9 mm to (47.1, 11.8)
- moved LEDR2 4.01 mm to (-19.7, 9.87)
- moved LEDR1 4.01 mm to (-16.4, 7.24)
- moved LEDR3 4.01 mm to (-23.3, 10.3)
- moved RGBLED1 4.01 mm to (-20.2, 9.43)
- moved TC2 1.85 mm to (98.4, 109.8)
Routing:
- net /GND: track 478.1 -> 533.7 mm
- net /IO13_TempData: track 30.4 -> 81.9 mm
- net /3V3: track 322.3 -> 371.2 mm, vias 8 -> 7
- net /IO12_LEDB: track 37.4 -> 34.0 mm
- net /IO14_LEDG: track 34.7 -> 32.3 mm
- net Net-(LEDR2-Pad1): track 2.45 -> 4.21 mm
- net /IO27_LEDR: track 28.7 -> 27.7 mm
Other:
- outline, holes or cut-outs redrawn

Commit message: revision 1.3
Parts:
- PC1: footprint Capacitor_SMD:CP_Elec_6.3x5.9 -> Capacitor_SMD:CP_Elec_10x12.5
- SMAJ18A1: footprint Diode_SMD:D_1210_3225Metric -> Diode_SMD:D_1210_3225Metric_Pad1.42x2.65mm_HandSolder
- UMW30N6: footprint Package_TO_SOT_SMD:TO-252-3_TabPin4 -> Package_TO_SOT_SMD:TO-252-2
- moved H5 159.4 mm to (10.0, 162.3), turned to 90 degrees
- moved H1 156.8 mm to (22.5, 166.0), turned to 90 degrees
- moved RST1 155.4 mm to (31.2, 167.9), turned to 0 degrees
- moved J2 153.5 mm to (55.1, 170.9), turned to 180 degrees
- moved H8 152.1 mm to (103.3, 162.1), turned to 90 degrees
- moved H2 151.9 mm to (91.0, 166.2), turned to 90 degrees
- moved ENR1 151.2 mm to (35.6, 166.1), turned to 90 degrees
- moved ESP_RST_C1 151.1 mm to (31.2, 164.8), turned to 180 degrees
- moved ESP_EN_C1 150.4 mm to (38.1, 166.1), turned to 90 degrees
- moved ESPC2 149.5 mm to (40.9, 166.1), turned to -90 degrees
- moved ESPC1 148.7 mm to (43.7, 166.0), turned to -90 degrees
- moved D1 148.1 mm to (69.1, 167.1), turned to 180 degrees
- moved LC8 145.6 mm to (84.0, 163.3), turned to -90 degrees
- moved LC6 144.9 mm to (81.3, 163.3), turned to -90 degrees
- moved AMS1117-5.0 144.1 mm to (76.2, 163.6), turned to -90 degrees
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Connections:
- UMW30N6 pad 1: Element -> /IO19_Gate
- UMW30N6 pad 2: /IO19_Gate -> Element
Routing:
- net Element: track 4869.8 -> 4884.3 mm
- net /IO17_UD2TX_NexRX: track 74.2 -> 83.6 mm
- net /5V0: track 29.3 -> 38.3 mm
- net /GND: track 533.7 -> 528.9 mm, vias 17 -> 19
- net /IO16_UD2RX_NexTX: track 77.9 -> 81.4 mm
- net /IO19_Gate: track 60.5 -> 64.0 mm
- net Net-(5A1-Pad2): track 6.55 -> 7.78 mm
Other:
- board size 170.7 x 111.2 mm -> 111.2 x 170.7 mm
- board text added: "+"
- board text added: "revision 1.3"
- board text removed: "OLED PANEL"
- board text removed: "revision 1.2"

Commit message: revision 1.3
Parts:
- removed AMS1117-3.3: AMS1117-3.3, Package_TO_SOT_SMD:SOT-223-3_TabPin2
- removed AMS1117-5.0: AMS1117-5.0, Package_TO_SOT_SMD:SOT-223-3_TabPin2
- removed PD1: DSR1M, Diode_SMD:D_SOD-123F
- added PD33: DSR1M, Diode_SMD:D_SOD-123F, B.Cu at (72.1, 148.3)
- added PD50: DSR1M, Diode_SMD:D_SOD-123F, B.Cu at (72.9, 150.9)
- added ZLDO1117-3.3: ZLDO1117-3.3, Package_TO_SOT_SMD:SOT-223-3_TabPin2 Reversed, B.Cu at (67.6, 159.6)
- added ZLDO1117-5.0: ZLDO1117-5.0, Package_TO_SOT_SMD:SOT-223-3_TabPin2 Reversed, B.Cu at (76.2, 163.8)
- moved PR2 1.98 mm to (64.0, 144.6)
- moved PR1 1.98 mm to (67.4, 144.5)
- turned LC1 to 180 degrees
- turned LC3 to 180 degrees
- turned LC5 to 180 degrees
- turned LC7 to 180 degrees
Routing:
- net /GND: track 528.9 -> 532.4 mm, vias 19 -> 20
- net /IO15_TempData: track 237.9 -> 234.4 mm
- net /IO19_Gate: track 64.0 -> 66.7 mm
- net /3V3: track 371.5 -> 369.0 mm
- net /5V0: track 38.3 -> 35.9 mm
- net Element: track 4884.3 -> 4886.3 mm
- net /VIN-D: track 50.2 -> 49.1 mm
- net VccDiv: track 51.0 -> 50.2 mm
- net /IO17_UD2TX_NexRX: track 83.6 -> 83.1 mm

Commit message: revision update
Parts:
- ZLDO1117-3.3, ZLDO1117-5.0: footprint Package_TO_SOT_SMD:SOT-223-3_TabPin2 Reversed -> Package_TO_SOT_SMD:SOT-223-3_TabPin2
- moved D1 22.6 mm to (87.7, 154.2), turned to -90 degrees
- moved LC8 7.41 mm to (90.7, 160.2)
- moved LC6 7.41 mm to (88.0, 160.2)
- moved LC5 4.90 mm to (80.3, 157.8), turned to 0 degrees
- moved LC7 4.82 mm to (80.4, 154.6), turned to 0 degrees
- moved ZLDO1117-5.0 4.82 mm to (81.0, 163.8)
- moved LC2 2.99 mm to (59.9, 155.9)
- moved LC4 2.31 mm to (59.9, 153.1)
- moved HR1 0.57 mm to (58.1, 150.7)
- turned LC1 to 0 degrees
- turned LC3 to 0 degrees
Routing:
- net Net-(D1-Pad2): track 22.0 -> 49.7 mm
- net /3V3: track 369.0 -> 350.5 mm, vias 7 -> 5
- net /GND: track 532.4 -> 523.2 mm, vias 20 -> 21
- net /IO15_TempData: track 234.4 -> 229.8 mm
- net /VIN-D: track 49.1 -> 47.0 mm
- net VccDiv: track 50.2 -> 49.2 mm
- net /IO19_Gate: track 66.7 -> 65.9 mm
- net /5V0: track 35.9 -> 36.5 mm
- added copper zone on B.Cu, net /3V3
- added copper zone on B.Cu, net /5V0
- added copper zone on B.Cu, net Element
Other:
- board text removed: "ESP32 & NEXTION version"

Commit message: revision update
Added some HiRes cool phtoos
Parts:
- removed PD33: DSR1M, Diode_SMD:D_SOD-123F
- added G***: LOGO, AeonLabs Logosy:CE Ready Small Logo, F.Cu at (103.2, 39.7)
- added G***: LOGO, AeonLabs Logosy:pcbWay Logo Collab, F.Cu at (-18.1, 78.5)
- added G***: LOGO, AeonLabs Logosy:CE Ready Small Logo, B.Cu at (103.9, 40.2)
- moved H7 139.5 mm to (10.3, 9.65), turned to 0 degrees
- moved H10 139.3 mm to (103.1, 113.5), turned to 0 degrees
- moved PD50 1.77 mm to (74.0, 152.3), turned to 90 degrees
- moved LMT1 0.36 mm to (10.6, 97.7)
- moved H9 0.30 mm to (10.2, 113.6), turned to 0 degrees
- turned SMAJ18A1 to 90 degrees
Connections:
- LC1 pad 2: /VIN-D -> /5V0
- LC3 pad 2: /VIN-D -> /5V0
- SMAJ18A1 pad 1: /GND -> Element
- SMAJ18A1 pad 2: Element -> /GND
- ZLDO1117-3.3 pad 3: /VIN-D -> /5V0
Routing:
- net Element: track 4886.3 -> 2301.4 mm
- net /5V0: track 36.5 -> 63.5 mm
- net /VIN-D: track 47.0 -> 35.5 mm
Other:
- outline, holes or cut-outs redrawn
- board text added: "revision 1.4"
- board text removed: "revision 1.3"

Commit message: rev. 2.0
added ON/OFF switch
Parts:
- removed CRX1: CRX, TestPoint:TestPoint_Pad_1.0x1.0mm
- removed CRX2: CRX2, TestPoint:TestPoint_Pad_1.0x1.0mm
- removed CTX1: CTX, TestPoint:TestPoint_Pad_1.0x1.0mm
- removed CTX2: CTX2, TestPoint:TestPoint_Pad_1.0x1.0mm
- removed LC5, LC6: 22uF, Capacitor_SMD:C_1206_3216Metric_Pad1.33x1.80mm_HandSolder
- removed LC7, LC8: 100nF, Capacitor_SMD:C_1206_3216Metric_Pad1.33x1.80mm_HandSolder
- removed ZLDO1117-3.3: ZLDO1117-3.3, Package_TO_SOT_SMD:SOT-223-3_TabPin2
- removed ZLDO1117-5.0: ZLDO1117-5.0, Package_TO_SOT_SMD:SOT-223-3_TabPin2
- added 0.7A1: Polyfuse, Fuse:Fuse_1206_3216Metric, B.Cu at (52.1, 161.6)
- added AC1: 22uF, Capacitor_SMD:C_0805_2012Metric_Pad1.18x1.45mm_HandSolder, B.Cu at (63.3, 161.8)
- added AC2: 4.7uF, Capacitor_SMD:C_0805_2012Metric_Pad1.18x1.45mm_HandSolder, B.Cu at (66.0, 157.4)
- added AMS1117-5.0S1: AMS1117-5.0S, Package_TO_SOT_SMD:SOT-223-3_TabPin2, B.Cu at (80.3, 164.2)
- added AR1: 3V3=1K5, Resistor_SMD:R_0805_2012Metric_Pad1.20x1.40mm_HandSolder, B.Cu at (68.8, 164.8)
- added AR2: 3V3=470R, Resistor_SMD:R_0805_2012Metric_Pad1.20x1.40mm_HandSolder, B.Cu at (68.7, 160.6)
- added AU1: AUR9718x_DFN_3x3mm_6_pin, Package_DFN_QFN:AUR9718 3x3mm 6 pin, B.Cu at (66.0, 160.6)
- added ML1: 3.3uF, Inductor_SMD:L_1210_3225Metric, B.Cu at (66.0, 165.3)
- added S1: DS04-254-1-01BK-SMT, AeonLabs:Side Switch 3pin 5A, B.Cu at (1.11, 134.3)
- added Sign-PbFree: , OLIMEX_LOGOs-FP:LOGO_PBFREE, F.Cu at (109.0, 82.3)
- added Sign-RecycleBin: , OLIMEX_LOGOs-FP:LOGO_RECYCLEBIN_1, F.Cu at (105.5, 84.5)
- added Sign-RoHS: , OLIMEX_LOGOs-FP:LOGO_ROHS_1, F.Cu at (108.6, 73.4)
- added TP1: VIN, TestPoint:TestPoint_Pad_D1.0mm, B.Cu at (62.8, 157.4)
- added TP2: VOut, TestPoint:TestPoint_Pad_D1.0mm, B.Cu at (63.0, 166.7)
- added TP3: GND, TestPoint:TestPoint_Pad_D1.0mm, B.Cu at (63.9, 151.5)
- 5A1: moved to F.Cu
- moved G*** 93.7 mm to (104.0, 66.0), turned to -90 degrees
- moved 5A1 76.3 mm to (15.9, 145.0), turned to -90 degrees
- moved D1 36.6 mm to (51.2, 157.5), turned to 180 degrees
- moved LC2 19.0 mm to (78.7, 158.5)
- moved LC4 18.9 mm to (78.6, 156.0)
- moved LC3 17.1 mm to (84.2, 156.1), turned to 180 degrees
- moved LC1 17.0 mm to (84.2, 158.5), turned to 180 degrees
- moved G*** 15.2 mm to (14.7, 44.0), turned to -90 degrees
- moved LEDR1 9.42 mm to (3.62, 150.2), turned to -90 degrees
- moved LEDR2 6.32 mm to (6.59, 150.3), turned to -90 degrees
- moved G*** 6.30 mm to (105.9, 45.4), turned to 90 degrees
- moved RGBLED1 5.92 mm to (6.32, 140.2)
- moved PR1 3.21 mm to (67.2, 147.7)
- moved PR2 3.21 mm to (63.8, 147.8)
- moved LEDR3 2.07 mm to (9.32, 150.3), turned to -90 degrees
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Connections:
- net /GND renamed GND
- D1 pad 1: /VIN-D -> VIN_DC
- D1 pad 2: Net-(D1-Pad2) -> Net-(0.7A1-Pad1)
- ENR1 pad 1: /3V3 -> 3V3
- ESP32-WROOM32 pad 10: unconnected-(ESP32-WROOM32-Pad10) -> /IO10_LEDG
- ESP32-WROOM32 pad 11: unconnected-(ESP32-WROOM32-Pad11) -> /IO26_LEDR
- ESP32-WROOM32 pad 12: /IO27_LEDR -> unconnected-(ESP32-WROOM32-Pad12)
- ESP32-WROOM32 pad 13: /IO14_LEDG -> unconnected-(ESP32-WROOM32-Pad13)
- ESP32-WROOM32 pad 2: /3V3 -> 3V3
- ESPC1 pad 1: /3V3 -> 3V3
- ESPC2 pad 1: /3V3 -> 3V3
- J1 pad 1: Net-(5A1-Pad2) -> Net-(J1-Pad1)
- J11 pad 1: /5V0 -> 5V0
- J2 pad 1: Net-(D1-Pad2) -> Net-(0.7A1-Pad2)
- J2 pad 3: Net-(CRX1-Pad1) -> /IO01TX
- J2 pad 4: Net-(CTX1-Pad1) -> /IO03RX
- LC1 pad 2: /5V0 -> VIN_DC
- LC2 pad 1: /3V3 -> 5V0
- LC3 pad 2: /5V0 -> VIN_DC
- LC4 pad 1: /3V3 -> 5V0
- LEDR2 pad 2: /IO14_LEDG -> /IO10_LEDG
- LEDR3 pad 2: /IO27_LEDR -> /IO26_LEDR
- LMT1 pad 1: /3V3 -> 3V3
- LMT2 pad 1: /3V3 -> 3V3
- PD50 pad 1: /VIN-D -> VIN_DC
- PR1 pad 1: /VIN-D -> VIN_DC
- TC1 pad 1: /3V3 -> 3V3
- TC2 pad 1: /3V3 -> 3V3
Routing:
- net /3V3: track 350.5 -> 0.00 mm, vias 5 -> 0
- net 3V3: track 0.00 -> 347.1 mm, vias 0 -> 6
- net Net-(J1-Pad1): track 0.00 -> 93.8 mm, vias 0 -> 1
- net Element: track 2301.4 -> 2389.3 mm, vias 5 -> 6
- net /5V0: track 63.5 -> 0.00 mm, vias 1 -> 0
- net 5V0: track 0.00 -> 56.5 mm, vias 0 -> 2
- net Net-(D1-Pad2): track 49.7 -> 0.00 mm, vias 2 -> 0
- net VIN_DC: track 0.00 -> 47.8 mm, vias 0 -> 2
- net /VIN-D: track 35.5 -> 0.00 mm, vias 2 -> 0
- net /IO14_LEDG: track 32.3 -> 0.00 mm, vias 2 -> 0
- net /IO10_LEDG: track 0.00 -> 30.9 mm, vias 0 -> 2
- net /IO27_LEDR: track 27.7 -> 0.00 mm, vias 2 -> 0
- net /IO26_LEDR: track 0.00 -> 26.5 mm, vias 0 -> 2
- net /IO03RX: track 20.8 -> 40.9 mm
- net /IO01TX: track 18.4 -> 38.5 mm, vias 0 -> 2
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- added copper zone on B.Cu, net 5V0
- removed copper zone on B.Cu, net /3V3
- removed copper zone on B.Cu, net /5V0
Other:
- copper layers 2 -> 6
- board text added: "3V3"
- board text added: "5V0"
- board text added: "DC2DC [0.8V to Vin] step down"
- board text added: "GND"
- board text added: "V-IN"
- board text added: "V-OUT"
- board text added: "revision 2.0"
- board text removed: "revision 1.4"
