File: ESP32 NEXTION/HotPlate.kicad_sch (KiCad schematic)
At the start: 56 parts, among them J1 Barrel_Jack_Switch, J11 Conn_01x04_Male, J2 Conn_01x08_Male

Commit message: revision 1.3
Parts:
- PC1: footprint Capacitor_SMD:CP_Elec_6.3x5.9 -> Capacitor_SMD:CP_Elec_10x12.5
- SMAJ18A1: footprint Diode_SMD:D_1210_3225Metric -> Diode_SMD:D_1210_3225Metric_Pad1.42x2.65mm_HandSolder
- UMW30N6: footprint Package_TO_SOT_SMD:TO-252-3_TabPin4 -> Package_TO_SOT_SMD:TO-252-2
Connections:
- net Element: now also UMW30N6.2 (G); no longer UMW30N6.1 (D)
- net IO19_Gate: now also UMW30N6.1 (D); no longer UMW30N6.2 (G)
Other:
- moved on the sheet: HR1, UMW30N6
Changed lines of the file:
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@@
   (junction (at 54.864 22.86) (diameter 0) (color 0 0 0 0)
   )
-  (junction (at 268.478 75.184) (diameter 0) (color 0 0 0 0)
-  )
   (junction (at 170.942 36.576) (diameter 0) (color 0 0 0 0)
   )
@@
   (junction (at 197.104 63.246) (diameter 0) (color 0 0 0 0)
   )
-  (junction (at 256.794 67.564) (diameter 0) (color 0 0 0 0)
-  )
   (junction (at 32.004 37.084) (diameter 0) (color 0 0 0 0)
   )
@@
   )
   (junction (at 82.296 47.244) (diameter 0) (color 0 0 0 0)
+  )
+  (junction (at 262.382 70.104) (diameter 0) (color 0 0 0 0)
   )
   (junction (at 263.144 59.944) (diameter 0) (color 0 0 0 0)
@@
   (no_connect (at 70.104 87.884))
   (no_connect (at 70.104 92.964))
-  (wire (pts (xy 256.794 75.184) (xy 268.478 75.184))
-    (stroke (width 0) (type default) (color 0 0 0 0))
-  )
   (polyline (pts (xy 192.532 134.62) (xy 192.532 114.046))
     (stroke (width 0) (type default) (color 0 0 0 0))
@@
     (stroke (width 0) (type default) (color 0 0 0 0))
   )
+  (wire (pts (xy 273.558 70.104) (xy 273.558 74.422))
+    (stroke (width 0) (type default) (color 0 0 0 0))
+  )
   (wire (pts (xy 251.46 140.97) (xy 251.46 143.764))
     (stroke (width 0) (type default) (color 0 0 0 0))
@@
     (stroke (width 0) (type default) (color 0 0 0 0))
   )
-  (wire (pts (xy 268.478 72.644) (xy 268.478 75.184))
-    (stroke (width 0) (type default) (color 0 0 0 0))
-  )
   (polyline (pts (xy 239.014 164.846) (xy 283.972 164.846))
     (stroke (width 0) (type default) (color 0 0 0 0))
@@
     (stroke (width 0) (type default) (color 0 0 0 0))
   )
+  (wire (pts (xy 254 70.104) (xy 254 74.422))
+    (stroke (width 0) (type default) (color 0 0 0 0))
+  )
   (wire (pts (xy 257.048 150.368) (xy 262.128 150.368))
     (stroke (width 0) (type default) (color 0 0 0 0))
@@
     (stroke (width 0) (type default) (color 0 0 0 0))
   )
-  (wire (pts (xy 250.444 67.564) (xy 256.794 67.564))
-    (stroke (width 0) (type default) (color 0 0 0 0))
-  )
   (wire (pts (xy 248.412 146.304) (xy 251.46 146.304))
     (stroke (width 0) (type default) (color 0 0 0 0))
@@
     (stroke (width 0) (type default) (color 0 0 0 0))
   )
+  (wire (pts (xy 254 74.422) (xy 273.558 74.422))
+    (stroke (width 0) (type default) (color 0 0 0 0))
+  )
   (wire (pts (xy 268.478 59.944) (xy 268.478 62.484))
     (stroke (width 0) (type default) (color 0 0 0 0))
@@
     (stroke (width 0) (type default) (color 0 0 0 0))
   )
+  (wire (pts (xy 262.382 70.104) (xy 263.398 70.104))
+    (stroke (width 0) (type default) (color 0 0 0 0))
+  )
+  (wire (pts (xy 262.382 65.024) (xy 262.382 70.104))
+    (stroke (width 0) (type default) (color 0 0 0 0))
+  )
   (wire (pts (xy 254.254 35.306) (xy 254.254 39.116))
     (stroke (width 0) (type default) (color 0 0 0 0))
@@
     (stroke (width 0) (type default) (color 0 0 0 0))
   )
+  (wire (pts (xy 261.62 70.104) (xy 262.382 70.104))
+    (stroke (width 0) (type default) (color 0 0 0 0))
+  )
   (wire (pts (xy 27.178 148.336) (xy 45.974 148.336))
     (stroke (width 0) (type default) (color 0 0 0 0))
@@
     (stroke (width 0) (type default) (color 0 0 0 0))
   )
-  (wire (pts (xy 268.478 75.184) (xy 268.478 75.692))
-    (stroke (width 0) (type default) (color 0 0 0 0))
-  )
   (wire (pts (xy 71.882 150.876) (xy 65.024 150.876))
     (stroke (width 0) (type default) (color 0 0 0 0))
@@
   )
   (wire (pts (xy 203.454 68.326) (xy 197.104 68.326))
-    (stroke (width 0) (type default) (color 0 0 0 0))
-  )
-  (wire (pts (xy 256.794 67.564) (xy 260.858 67.564))
     (stroke (width 0) (type default) (color 0 0 0 0))
   )
@@
     (effects (font (size 1.27 1.27)) (justify left bottom))
   )
-  (label "GND" (at 268.478 75.692 0)
+  (label "GND" (at 262.382 65.024 0)
     (effects (font (size 1.27 1.27)) (justify left bottom))
   )
@@
     (effects (font (size 1.27 1.27)) (justify left bottom))
   )
-  (label "IO19_Gate" (at 250.444 67.564 180)
+  (label "IO19_Gate" (at 254 70.104 180)
     (effects (font (size 1.27 1.27)) (justify right bottom))
   )
@@
       (effects (font (size 1.27 1.27)) (justify left))
     )
-    (property "Footprint" "Capacitor_SMD:CP_Elec_6.3x5.9" (id 2) (at 236.1692 30.48 0)
+    (property "Footprint" "Capacitor_SMD:CP_Elec_10x12.5" (id 2) (at 236.1692 30.48 0)
       (effects (font (size 1.27 1.27)) hide)
     )
@@
       (effects (font (size 1.27 1.27)) (justify right))
     )
-    (property "Footprint" "Diode_SMD:D_1210_3225Metric" (id 2) (at 226.568 27.178 0)
+    (property "Footprint" "Diode_SMD:D_1210_3225Metric_Pad1.42x2.65mm_HandSolder" (id 2) (at 226.568 27.178 0)
       (effects (font (size 1.27 1.27)) hide)
     )
@@
     (pin "2")
   )
-  (symbol (lib_id "Device:R") (at 256.794 71.374 0) (unit 1)
-    (in_bom yes) (on_board yes)
-    (property "Reference" "HR1" (id 0) (at 258.318 73.152 0)
-      (effects (font (size 1.27 1.27)) (justify left))
-    )
-    (property "Value" "10K" (id 1) (at 258.064 70.612 0)
-      (effects (font (size 1.27 1.27)) (justify left))
-    )
-    (property "Footprint" "Capacitor_SMD:C_1206_3216Metric_Pad1.33x1.80mm_HandSolder" (id 2) (at 255.016 71.374 90)
-      (effects (font (size 1.27 1.27)) hide)
-    )
-    (property "Datasheet" "~" (id 3) (at 256.794 71.374 0)
+  (symbol (lib_id "Device:R") (at 257.81 70.104 90) (unit 1)
+    (in_bom yes) (on_board yes)
+    (property "Reference" "HR1" (id 0) (at 258.064 68.326 0)
+      (effects (font (size 1.27 1.27)) (justify left))
+    )
+    (property "Value" "10K" (id 1) (at 256.032 68.58 0)
+      (effects (font (size 1.27 1.27)) (justify left))
+    )
+    (property "Footprint" "Capacitor_SMD:C_1206_3216Metric_Pad1.33x1.80mm_HandSolder" (id 2) (at 257.81 71.882 90)
+      (effects (font (size 1.27 1.27)) hide)
+    )
+    (property "Datasheet" "~" (id 3) (at 257.81 70.104 0)
       (effects (font (size 1.27 1.27)) hide)
     )
@@
     (pin "2")
   )
-  (symbol (lib_id "Device:Q_NMOS_DGS") (at 265.938 67.564 0) (unit 1)
-    (in_bom yes) (on_board yes) (fields_autoplaced)
-    (property "Reference" "UMW30N6" (id 0) (at 271.145 66.6555 0)
-      (effects (font (size 1.27 1.27)) (justify left))
-    )
-    (property "Value" "HM" (id 1) (at 271.145 69.4306 0)
-      (effects (font (size 1.27 1.27)) (justify left))
-    )
-    (property "Footprint" "Package_TO_SOT_SMD:TO-252-3_TabPin4" (id 2) (at 271.018 65.024 0)
-      (effects (font (size 1.27 1.27)) hide)
-    )
-    (property "Datasheet" "~" (id 3) (at 265.938 67.564 0)
+  (symbol (lib_id "Device:Q_NMOS_DGS") (at 268.478 67.564 270) (unit 1)
+    (in_bom yes) (on_board yes)
+    (property "Reference" "UMW30N6" (id 0) (at 278.13 67.056 90))
+    (property "Value" "HM" (id 1) (at 277.622 69.088 90))
+    (property "Footprint" "Package_TO_SOT_SMD:TO-252-2" (id 2) (at 271.018 72.644 0)
+      (effects (font (size 1.27 1.27)) hide)
+    )
+    (property "Datasheet" "~" (id 3) (at 268.478 67.564 0)
       (effects (font (size 1.27 1.27)) hide)
     )
@@
     )
     (path "/04997c0e-f533-4da3-8aed-3484d2569925"
-      (reference "PC1") (unit 1) (value "100uF") (footprint "Capacitor_SMD:CP_Elec_6.3x5.9")
+      (reference "PC1") (unit 1) (value "100uF") (footprint "Capacitor_SMD:CP_Elec_10x12.5")
     )
     (path "/43452d5b-ba44-4473-b7ed-b0e4c7902559"
@@
     )
     (path "/737c3eb0-edd7-42a7-b782-07a107f00a56"
-      (reference "SMAJ18A1") (unit 1) (value "SMAJ18A") (footprint "Diode_SMD:D_1210_3225Metric")
+      (reference "SMAJ18A1") (unit 1) (value "SMAJ18A") (footprint "Diode_SMD:D_1210_3225Metric_Pad1.42x2.65mm_HandSolder")
     )
     (path "/8fb3f598-be1a-4928-9caf-76ce6e9fe6e3"
@@
     )
     (path "/ca0239ea-7847-4675-adb8-634cbeec5b9a"
-      (reference "UMW30N6") (unit 1) (value "HM") (footprint "Package_TO_SOT_SMD:TO-252-3_TabPin4")
-    )
-  )
+      (reference "UMW30N6") (unit 1) (value "HM") (footprint "Package_TO_SOT_SMD:TO-252-2")
+    )
+  )

Commit message: revision 1.3
Parts:
- added PD33: DSR1M, Diode_SMD:D_SOD-123F, symbol Device:D
- ZLDO1117-3.3: renamed from AMS1117-3.3; value AMS1117-3.3 -> ZLDO1117-3.3; footprint Package_TO_SOT_SMD:SOT-223-3_TabPin2 -> Package_TO_SOT_SMD:SOT-223-3_TabPin2 Reversed
- ZLDO1117-5.0: renamed from AMS1117-5.0; value AMS1117-5.0 -> ZLDO1117-5.0; footprint Package_TO_SOT_SMD:SOT-223-3_TabPin2 -> Package_TO_SOT_SMD:SOT-223-3_TabPin2 Reversed
- renumbered PD1 to PD50
Connections:
- net Element: now also PD33.2 (A)
- net VIN-D: now also PD33.1 (K)
Other:
- moved on the sheet: LEDR1, LEDR2, LEDR3, RGBLED1

Commit message: revision update
Parts:
- ZLDO1117-3.3, ZLDO1117-5.0: footprint Package_TO_SOT_SMD:SOT-223-3_TabPin2 Reversed -> Package_TO_SOT_SMD:SOT-223-3_TabPin2
Changed lines of the file:
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@@
       (effects (font (size 1.27 1.27)) (justify left))
     )
-    (property "Footprint" "Package_TO_SOT_SMD:SOT-223-3_TabPin2 Reversed" (id 2) (at 131.064 60.452 0)
+    (property "Footprint" "Package_TO_SOT_SMD:SOT-223-3_TabPin2" (id 2) (at 131.064 60.452 0)
       (effects (font (size 1.27 1.27)) hide)
     )
@@
       (effects (font (size 1.27 1.27)) (justify left))
     )
-    (property "Footprint" "Package_TO_SOT_SMD:SOT-223-3_TabPin2 Reversed" (id 2) (at 145.796 28.956 0)
+    (property "Footprint" "Package_TO_SOT_SMD:SOT-223-3_TabPin2" (id 2) (at 145.796 28.956 0)
       (effects (font (size 1.27 1.27)) hide)
     )
@@
     )
     (path "/eb63c3d5-07d6-4ad3-9fe3-e2c15774aca4"
-      (reference "ZLDO1117-3.3") (unit 1) (value "ZLDO1117-3.3") (footprint "Package_TO_SOT_SMD:SOT-223-3_TabPin2 Reversed")
+      (reference "ZLDO1117-3.3") (unit 1) (value "ZLDO1117-3.3") (footprint "Package_TO_SOT_SMD:SOT-223-3_TabPin2")
     )
     (path "/5cc29f4c-048d-4236-94d4-82c6ee8e1268"
-      (reference "ZLDO1117-5.0") (unit 1) (value "ZLDO1117-5.0") (footprint "Package_TO_SOT_SMD:SOT-223-3_TabPin2 Reversed")
-    )
-  )
+      (reference "ZLDO1117-5.0") (unit 1) (value "ZLDO1117-5.0") (footprint "Package_TO_SOT_SMD:SOT-223-3_TabPin2")
+    )
+  )

Commit message: revision update
Added some HiRes cool phtoos
Parts:
- removed PD33: DSR1M, Diode_SMD:D_SOD-123F, symbol Device:D
Connections:
- net 5V0: now also LC1.2, LC3.2, ZLDO1117-3.3.3 (VI)
- net Element: now also SMAJ18A1.1 (A1); no longer SMAJ18A1.2 (A2)
- net GND: now also SMAJ18A1.2 (A2); no longer SMAJ18A1.1 (A1)
- net VIN-D: no longer LC1.2, LC3.2, ZLDO1117-3.3.3 (VI)
Other:
- moved on the sheet: SMAJ18A1
Changed lines of the file:
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@@
   (junction (at 226.568 20.066) (diameter 0) (color 0 0 0 0)
-  )
-  (junction (at 250.444 20.066) (diameter 0) (color 0 0 0 0)
   )
   (junction (at 161.29 60.452) (diameter 0) (color 0 0 0 0)
@@
     (stroke (width 0) (type default) (color 0 0 0 0))
   )
-  (wire (pts (xy 250.698 20.066) (xy 250.444 20.066))
+  (wire (pts (xy 246.888 20.066) (xy 250.698 20.066))
     (stroke (width 0) (type default) (color 0 0 0 0))
   )
@@
     (stroke (width 0) (type default) (color 0 0 0 0))
   )
-  (wire (pts (xy 260.604 24.384) (xy 260.604 20.066))
-    (stroke (width 0) (type default) (color 0 0 0 0))
-  )
   (polyline (pts (xy 192.532 77.978) (xy 237.49 77.978))
     (stroke (width 0) (type default) (color 0 0 0 0))
   )
-  (wire (pts (xy 258.064 24.384) (xy 260.604 24.384))
-    (stroke (width 0) (type default) (color 0 0 0 0))
-  )
   (polyline (pts (xy 192.786 135.89) (xy 192.786 164.846))
     (stroke (width 0) (type default) (color 0 0 0 0))
@@
     (stroke (width 0) (type default) (color 0 0 0 0))
   )
-  (wire (pts (xy 250.444 20.066) (xy 250.444 24.384))
-    (stroke (width 0) (type default) (color 0 0 0 0))
-  )
   (wire (pts (xy 90.678 193.548) (xy 76.708 193.548))
     (stroke (width 0) (type default) (color 0 0 0 0))
@@
   )
   (wire (pts (xy 211.074 129.286) (xy 203.454 129.286))
-    (stroke (width 0) (type default) (color 0 0 0 0))
-  )
-  (wire (pts (xy 250.444 20.066) (xy 246.888 20.066))
     (stroke (width 0) (type default) (color 0 0 0 0))
   )
@@
     (effects (font (size 1.27 1.27)) (justify left bottom))
   )
-  (label "VIN-D" (at 186.436 36.576 0)
+  (label "5V0" (at 186.436 36.576 0)
     (effects (font (size 1.27 1.27)) (justify left bottom))
   )
@@
     (pin "2")
   )
-  (symbol (lib_id "Diode:ESD9B3.3ST5G") (at 226.568 27.178 90) (unit 1)
-    (in_bom yes) (on_board yes)
-    (property "Reference" "SMAJ18A1" (id 0) (at 228.6 18.542 90)
+  (symbol (lib_id "Diode:ESD9B3.3ST5G") (at 226.568 27.178 270) (unit 1)
+    (in_bom yes) (on_board yes)
+    (property "Reference" "SMAJ18A1" (id 0) (at 237.109 18.034 90)
       (effects (font (size 1.27 1.27)) (justify right))
     )
-    (property "Value" "SMAJ18A" (id 1) (at 229.362 16.256 90)
+    (property "Value" "SMAJ18A" (id 1) (at 236.347 16.002 90)
       (effects (font (size 1.27 1.27)) (justify right))
     )
@@
     (pin "3")
   )
-  (symbol (lib_id "Device:D") (at 254.254 24.384 180) (unit 1)
-    (in_bom yes) (on_board yes)
-    (property "Reference" "PD33" (id 0) (at 254.508 29.464 0))
-    (property "Value" "DSR1M" (id 1) (at 254.508 27.178 0))
-    (property "Footprint" "Diode_SMD:D_SOD-123F" (id 2) (at 254.254 24.384 0)
-      (effects (font (size 1.27 1.27)) hide)
-    )
-    (property "Datasheet" "~" (id 3) (at 254.254 24.384 0)
-      (effects (font (size 1.27 1.27)) hide)
-    )
-    (pin "1")
-    (pin "2")
-  )
   (symbol (lib_id "Device:C") (at 165.862 25.146 0) (unit 1)
     (in_bom yes) (on_board yes)
@@
       (reference "PC3") (unit 1) (value "1nF") (footprint "Capacitor_SMD:C_1206_3216Metric_Pad1.33x1.80mm_HandSolder")
     )
-    (path "/e1488c0d-62fb-423b-b706-0991ba3d49e1"
-      (reference "PD33") (unit 1) (value "DSR1M") (footprint "Diode_SMD:D_SOD-123F")
-    )
     (path "/e2b5dd16-d649-4f0f-b4ba-dca0c7f9e14e"

Commit message: rev. 2.0
added ON/OFF switch
Parts:
- removed CRX1: CRX, TestPoint:TestPoint_Pad_1.0x1.0mm, symbol Connector:TestPoint
- removed CRX2: CRX2, TestPoint:TestPoint_Pad_1.0x1.0mm, symbol Connector:TestPoint
- removed CTX1: CTX, TestPoint:TestPoint_Pad_1.0x1.0mm, symbol Connector:TestPoint
- removed CTX2: CTX2, TestPoint:TestPoint_Pad_1.0x1.0mm, symbol Connector:TestPoint
- removed LC5, LC6: 22uF, Capacitor_SMD:C_1206_3216Metric_Pad1.33x1.80mm_HandSolder, symbol Device:C
- removed LC7, LC8: 100nF, Capacitor_SMD:C_1206_3216Metric_Pad1.33x1.80mm_HandSolder, symbol Device:C
- removed ZLDO1117-5.0: ZLDO1117-5.0, Package_TO_SOT_SMD:SOT-223-3_TabPin2, symbol Regulator_Linear:AMS1117-5.0
- added 0.7A1: Polyfuse, Fuse:Fuse_1206_3216Metric, symbol Device:Polyfuse
- added AC1: 22uF, Capacitor_SMD:C_0805_2012Metric_Pad1.18x1.45mm_HandSolder, symbol Device:C
- added AC2: 4.7uF, Capacitor_SMD:C_0805_2012Metric_Pad1.18x1.45mm_HandSolder, symbol Device:C
- added AR1: 3V3=1K5, Resistor_SMD:R_0805_2012Metric_Pad1.20x1.40mm_HandSolder, symbol Device:R
- added AR2: 3V3=470R, Resistor_SMD:R_0805_2012Metric_Pad1.20x1.40mm_HandSolder, symbol Device:R
- added AU1: AUR9718x_DFN_3x3mm_6_pin, Package_DFN_QFN:AUR9718 3x3mm 6 pin, symbol Power_Management:AUR9718x_DFN_3x3mm_6_pin
- added ML1: 3.3uF, Inductor_SMD:L_1210_3225Metric, symbol Device:L
- added S1: DS04-254-1-01BK-SMT, AeonLabs:Side Switch 3pin 5A, symbol SMD DIP toggle switches:DS04-254-1-01BK-SMT
- added TP1: VIN, TestPoint:TestPoint_Pad_D1.0mm, symbol Connector:TestPoint
- added TP2: VOut, TestPoint:TestPoint_Pad_D1.0mm, symbol Connector:TestPoint
- added TP3: GND, TestPoint:TestPoint_Pad_D1.0mm, symbol Connector:TestPoint
- AMS1117-5.0S1: renamed from ZLDO1117-3.3; value ZLDO1117-3.3 -> AMS1117-5.0S
Connections:
- net 3V3: now also AC1.1, AR1.1, ML1.1, TP2.1; no longer AMS1117-5.0S1.2 (VO), LC2.1, LC4.1
- net 5V0: now also AMS1117-5.0S1.2 (VO), LC2.1, LC4.1, AC2.1, AU1.4 (VIN_SW), AU1.5 (VIN_A), AU1.6 (EN), TP1.1; no longer AMS1117-5.0S1.3 (VI), LC1.2, LC3.2
- net GND: now also AC1.2, AC2.2, AR2.2, AU1.2 (GND), TP3.1
- net IO01TX: now also J2.3 (Pin_3)
- net IO03RX: now also J2.4 (Pin_4)
- net IO10_LEDG: now reaches ESP32-WROOM32.10 (IO25)
- net IO10_LEDG: now also LEDR2.2
- net IO26_LEDR: now reaches ESP32-WROOM32.11 (IO26)
- net IO26_LEDR: now also LEDR3.2
- net at J1.1: now also S1.1B; no longer 5A1.2
- net at D1.2 (A): now also 0.7A1.1; no longer J2.1 (Pin_1)
- net IO14_LEDG: no longer names the net of ESP32-WROOM32.13 (IO14)
- net IO14_LEDG: no longer LEDR2.2
- net IO27_LEDR: no longer names the net of ESP32-WROOM32.12 (IO27)
- net IO27_LEDR: no longer LEDR3.2
- net VIN-D renamed VIN_DC
- net VIN_DC: now also AMS1117-5.0S1.3 (VI), LC1.2, LC3.2
- new net: 5A1.2, S1.1A
- new net: AR1.2, AR2.1, AU1.1 (FB)
- new net: AU1.3 (SW), ML1.2
- new net: 0.7A1.2, J2.1 (Pin_1)
- no-connect marks 19 -> 21
Other:
- note added: "1uF to 6.8uF"
- note added: "5V LDO and Filtering"
- note added: "VIN 2.7V to 5.5V"
- note added: "Vout=0.8x(1+R1/R2)"
- note removed: "3V3 LDO and Filtering"
- note removed: "5V0 LDO and Filtering"
- note removed: "Microcontroller"
- moved on the sheet: 5A1, AMS1117-5.0S1, BUZZER1, D1, ENR1, ESP32-WROOM32, ESPC1, ESPC2, ESPC4, ESP_EN_C1, ESP_RST_C1, H1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
